File: Hardware/SYNCHRO_Booster/SYNCHRO_Booster.kicad_sch (KiCad schematic)
At the start: 42 parts, among them IC1 L6203, J1 Conn_01x02_Pin, J2 Power_Input, J3 B4B-XH-A, J4 Messpunkt, SW1 SW_Push, SW2 SW_SPDT, U1 LM393P, U2 6N137, U3 6N137, U4 74LVC2G02

Commit message: Booster_Design_v1.0
Parts:
- added F1: MF-R185-2-99, SYNCHRO_Library:Fuse_Bourns_MF-R185, symbol Device:Fuse
Connections:
- net +5V: no longer J4.1 (Pin_1)
- net SENSE: now also J4.1 (Pin_1)
- net at SW2.2 (B), SW2.3 (C): now also F1.1; no longer J2.1 (Pin_1)
- new net: F1.2, J2.1 (Pin_1)
Other:
- moved on the sheet: SW2
