File: Hardware/SYNCHRO_Zentrale/SYNCHRO_Zentrale.kicad_pcb (KiCad board)
At the start: 2 copper layers, 0 parts

Commit message: hardware update push
Parts:
- added C1: 22uF, Capacitor_SMD:C_1210_3225Metric_Pad1.33x2.70mm_HandSolder, F.Cu at (44.9, 23.8)
- added C10: 10uF, Capacitor_SMD:C_1210_3225Metric_Pad1.33x2.70mm_HandSolder, F.Cu at (112.1, 88.9)
- added C11: 10uF, Capacitor_SMD:C_1210_3225Metric_Pad1.33x2.70mm_HandSolder, F.Cu at (101.9, 45.2)
- added C12: 22uF, Capacitor_SMD:C_1210_3225Metric_Pad1.33x2.70mm_HandSolder, F.Cu at (95.2, 34.7)
- added C2: 0.1uF, Capacitor_SMD:C_1206_3216Metric_Pad1.33x1.80mm_HandSolder, F.Cu at (37.4, 68.2)
- added C3: 1uF, Capacitor_SMD:C_1206_3216Metric_Pad1.33x1.80mm_HandSolder, F.Cu at (37.4, 71.5)
- added C4: 0.1uF, Capacitor_SMD:C_1206_3216Metric_Pad1.33x1.80mm_HandSolder, F.Cu at (37.4, 74.9)
- added C5: 10uF, Capacitor_SMD:C_1210_3225Metric_Pad1.33x2.70mm_HandSolder, F.Cu at (112.1, 64.8)
- added C6: 10uF, Capacitor_SMD:C_1210_3225Metric_Pad1.33x2.70mm_HandSolder, F.Cu at (121.9, 72.1)
- added C7: 100nF, Capacitor_SMD:C_1206_3216Metric_Pad1.33x1.80mm_HandSolder, F.Cu at (141.0, 34.3)
- added C8: 100nF, Capacitor_SMD:C_1206_3216Metric_Pad1.33x1.80mm_HandSolder, F.Cu at (141.0, 91.4)
- added C9: 10uF, Capacitor_SMD:C_1210_3225Metric_Pad1.33x2.70mm_HandSolder, F.Cu at (121.9, 82.3)
- added D1: PMEG3010ER, Diode_SMD:Nexperia_CFP3_SOD-123W, F.Cu at (101.7, 38.8)
- added D2: LED, LED_THT:LED_D5.0mm, F.Cu at (36.8, 25.4)
- added D3: LED, LED_THT:LED_D5.0mm, F.Cu at (36.8, 32.9)
- added D4: LED, LED_THT:LED_D5.0mm, F.Cu at (36.8, 40.3)
- added D5: LED, LED_THT:LED_D5.0mm, F.Cu at (36.8, 47.8)
- added D6: LED, LED_THT:LED_D5.0mm, F.Cu at (36.8, 55.3)
- added D7: LED, LED_THT:LED_D5.0mm, F.Cu at (36.8, 62.8)
- added IC1: MC74VHCT541ADWR2G, SYNCHRO_Library:SOIC127P1030X265-20N, F.Cu at (138.1, 99.7)
- added IC2: MC74VHCT541ADWR2G, SYNCHRO_Library:SOIC127P1030X265-20N, F.Cu at (138.1, 42.5)
- added IC3: AZ1117CH-3.3TRG1, SYNCHRO_Library:SOT230P700X180-4N, F.Cu at (95.2, 41.9)
- added J1: GSB22120RSKEU, SYNCHRO_Library:AMPHENOL_GSB22120RSKEU, F.Cu at (94.0, 56.2)
- added J10: 694106301002, SYNCHRO_Library:694106301002, F.Cu at (99.8, 73.7)
- added J2: B4B-XH-A_LF__SN_, SYNCHRO_Library:JST_B4B-XH-A_LF__SN_, F.Cu at (168.2, 49.6)
- added J3: B4B-XH-A_LF__SN_, SYNCHRO_Library:JST_B4B-XH-A_LF__SN_, F.Cu at (168.2, 64.8)
- added J4: B4B-XH-A_LF__SN_, SYNCHRO_Library:JST_B4B-XH-A_LF__SN_, F.Cu at (168.2, 80.0)
- added J5: B4B-XH-A_LF__SN_, SYNCHRO_Library:JST_B4B-XH-A_LF__SN_, F.Cu at (168.2, 95.3)
- added J6: B4B-XH-A_LF__SN_, SYNCHRO_Library:JST_B4B-XH-A_LF__SN_, F.Cu at (155.5, 95.3)
- added J7: B4B-XH-A_LF__SN_, SYNCHRO_Library:JST_B4B-XH-A_LF__SN_, F.Cu at (155.5, 80.1)
- added J8: B4B-XH-A_LF__SN_, SYNCHRO_Library:JST_B4B-XH-A_LF__SN_, F.Cu at (155.5, 64.8)
- added J9: B4B-XH-A_LF__SN_, SYNCHRO_Library:JST_B4B-XH-A_LF__SN_, F.Cu at (155.5, 49.6)
- added PS1: R-78E3.3-0.5, SYNCHRO_Library:CONV_R-78E3.3-0.5, F.Cu at (113.0, 71.4)
- added PS2: R-78E5.0-1.0, SYNCHRO_Library:R78E5010, F.Cu at (110.5, 83.8)
- added R1: 10k, Resistor_SMD:R_0805_2012Metric_Pad1.20x1.40mm_HandSolder, F.Cu at (27.6, 136.2)
- added R10: 220, Resistor_SMD:R_0805_2012Metric_Pad1.20x1.40mm_HandSolder, F.Cu at (37.1, 139.2)
- added R11: 220, Resistor_SMD:R_0805_2012Metric_Pad1.20x1.40mm_HandSolder, F.Cu at (37.1, 142.1)
- added R12: 470, Resistor_SMD:R_0805_2012Metric_Pad1.20x1.40mm_HandSolder, F.Cu at (37.1, 145.1)
- added R2: 10k, Resistor_SMD:R_0805_2012Metric_Pad1.20x1.40mm_HandSolder, F.Cu at (27.6, 139.2)
- added R3: 10k, Resistor_SMD:R_0805_2012Metric_Pad1.20x1.40mm_HandSolder, F.Cu at (27.6, 142.1)
- added R4: 10k, Resistor_SMD:R_0805_2012Metric_Pad1.20x1.40mm_HandSolder, F.Cu at (27.6, 145.1)
- added R5: 10k, Resistor_SMD:R_0805_2012Metric_Pad1.20x1.40mm_HandSolder, F.Cu at (32.3, 136.2)
- added R6: 10k, Resistor_SMD:R_0805_2012Metric_Pad1.20x1.40mm_HandSolder, F.Cu at (32.3, 139.2)
- added R7: 220, Resistor_SMD:R_0805_2012Metric_Pad1.20x1.40mm_HandSolder, F.Cu at (32.3, 142.1)
- added R8: 220, Resistor_SMD:R_0805_2012Metric_Pad1.20x1.40mm_HandSolder, F.Cu at (32.3, 145.1)
- added R9: 220, Resistor_SMD:R_0805_2012Metric_Pad1.20x1.40mm_HandSolder, F.Cu at (37.1, 136.2)
- added SW1: SW_Push, Button_Switch_THT:SW_PUSH_6mm, F.Cu at (27.2, 119.7)
- added SW2: SW_Push, Button_Switch_THT:SW_PUSH_6mm, F.Cu at (27.2, 128.2)
- added SW3: SW_Push, Button_Switch_THT:SW_PUSH_6mm, F.Cu at (44.2, 101.0)
- added SW4: SW_Push, Button_Switch_THT:SW_PUSH_6mm, F.Cu at (44.2, 109.6)
- added SW5: SW_Push, Button_Switch_THT:SW_PUSH_6mm, F.Cu at (44.2, 118.1)
- added SW6: SW_Push, Button_Switch_THT:SW_PUSH_6mm, F.Cu at (44.2, 126.7)
- added U1: ESP32-S3-WROOM-1-N8R8, SYNCHRO_Library:ESP32S3WROOM1N8R8, F.Cu at (116.9, 38.6)
Routing:
- net /DCC_Signal_A_1: track 0.00 -> 109.2 mm
- net /DCC_Signal_A_2: track 0.00 -> 89.5 mm
- net /DCC_Signal_A_8: track 0.00 -> 73.9 mm
- net /DCC_Signal_B_4: track 0.00 -> 70.4 mm
- net /DCC_Signal_A_3: track 0.00 -> 69.8 mm
- net /DCC_Signal_B_5: track 0.00 -> 61.2 mm
- net /DCC_Signal_A_7: track 0.00 -> 56.8 mm
- net /DCC_Signal_B_3: track 0.00 -> 56.4 mm
- net /DCC_Signal_B_6: track 0.00 -> 48.8 mm
- net /DCC_Signal_B_2: track 0.00 -> 42.4 mm
- net /DCC_Signal_A_4: track 0.00 -> 41.2 mm
- net /DCC_Signal_A_6: track 0.00 -> 39.6 mm
- net Net-(J10-POWER): track 0.00 -> 34.8 mm
- net /DCC_Signal_B_7: track 0.00 -> 32.0 mm
- net /DCC_Signal_B_1: track 0.00 -> 28.5 mm
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- added copper zone on B.Cu, net +5V_Z
- added copper zone on F.Cu, net GND
Other:
- board outline added: 165.1 x 127 mm

Commit message: Zentrale Layout V1.0 finalisierung
Parts:
- added REF**: MountingHole_3.2mm_M3, MountingHole:MountingHole_3.2mm_M3, F.Cu at (170.2, 36.2)
- added REF**: MountingHole_3.2mm_M3, MountingHole:MountingHole_3.2mm_M3, F.Cu at (96.5, 103.5)
- added REF**: MountingHole_3.2mm_M3, MountingHole:MountingHole_3.2mm_M3, F.Cu at (170.2, 117.5)
- moved R1 123.6 mm to (98.0, 34.7), turned to 90 degrees
- moved SW2 119.3 mm to (125.7, 61.0), turned to 180 degrees
- moved R2 117.5 mm to (118.5, 64.8)
- moved R6 108.8 mm to (139.1, 118.1), turned to -90 degrees
- moved D5 107.2 mm to (127.0, 105.7), turned to 90 degrees
- moved D4 105.3 mm to (119.4, 105.7), turned to 90 degrees
- moved D2 104.8 mm to (104.1, 105.7), turned to 90 degrees
- moved D3 104.5 mm to (111.8, 105.7), turned to 90 degrees
- moved SW1 103.4 mm to (109.1, 56.5)
- moved R4 103.0 mm to (127.0, 118.1), turned to -90 degrees
- moved R10 99.0 mm to (128.0, 100.0)
- moved R8 92.2 mm to (112.8, 100.0)
- moved R9 90.8 mm to (120.4, 100.0)
- moved SW6 87.7 mm to (131.4, 116.9), turned to 90 degrees
- moved R11 84.7 mm to (102.2, 88.0), turned to -90 degrees
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Connections:
- U1 pad 10: /IO17 -> unconnected-(U1-IO17-Pad10)
- U1 pad 11: /IO18 -> unconnected-(U1-IO18-Pad11)
- U1 pad 22: /IO14 -> unconnected-(U1-IO14-Pad22)
- U1 pad 23: /IO21 -> unconnected-(U1-IO21-Pad23)
- U1 pad 8: /IO15 -> unconnected-(U1-IO15-Pad8)
- U1 pad 9: /IO16 -> unconnected-(U1-IO16-Pad9)
Routing:
- net +3.3V: track 12.6 -> 183.7 mm, vias 0 -> 2
- net GND: track 0.00 -> 169.2 mm, vias 0 -> 17
- net /IO7: track 0.00 -> 108.8 mm, vias 0 -> 1
- net /IO8: track 0.00 -> 92.2 mm, vias 0 -> 1
- net /IO6: track 0.00 -> 87.1 mm, vias 0 -> 1
- net /IO9: track 0.00 -> 85.6 mm, vias 0 -> 1
- net /Z_Out_DCC_Signal_A: track 8.89 -> 85.8 mm, vias 0 -> 2
- net /IO10: track 0.00 -> 61.2 mm, vias 0 -> 2
- net /IO11: track 0.00 -> 57.4 mm, vias 0 -> 2
- net /IO13: track 0.00 -> 55.9 mm, vias 0 -> 2
- net /IO12: track 0.00 -> 53.7 mm, vias 0 -> 2
- net /Z_Out_DCC_Signal_B: track 8.89 -> 34.2 mm, vias 0 -> 2
- net +5V_Z: track 16.2 -> 40.4 mm
- net Net-(U1-IO0): track 0.00 -> 22.7 mm
- net Net-(U1-3V3): track 0.00 -> 14.9 mm
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Other:
- board size 165.1 x 127 mm -> 84.5 x 90.2 mm
- board text added: "+3.3V"
- board text added: "+5V"
