File: Hardware/SYNCHRO_Zentrale/SYNCHRO_Zentrale.kicad_sch (KiCad schematic)
At the start: 12 parts, among them J1 GSB22120RSKEU, SW1 SW_Push, SW2 SW_Push, U1 ESP32-S3-WROOM-1-N8R8

Commit message: SYNCHRO Zentrale design backup
Parts:
- added C6: 10uF, Capacitor_SMD:C_1210_3225Metric_Pad1.33x2.70mm_HandSolder, symbol Device:C
- added C7, C8: 100nF, Capacitor_SMD:C_1206_3216Metric_Pad1.33x1.80mm_HandSolder, symbol Device:C
- added D1: SMAJ5.0A, SYNCHRO_Library:DIOM5226X243N, symbol SYNCHRO_Library:SMAJ5.0A
- added IC1, IC2: MC74VHCT541ADWR2G, SYNCHRO_Library:SOIC127P1030X265-20N, symbol SYNCHRO_Library:MC74VHCT541ADWR2G
- added J2, J3, J4, J5, J6, J7, J8, J9: B4B-XH-A_LF__SN_, SYNCHRO_Library:JST_B4B-XH-A_LF__SN_, symbol SYNCHRO_Library:B4B-XH-A_LF__SN_
Connections:
- net +3.3V: now also C6.1
- net GND: now also C6.2, C7.2, C8.2, D1.2 (A), IC1.1 (~{OE1}), IC1.10 (GND), IC1.19 (~{OE2}), IC2.1 (~{OE1}), IC2.10 (GND), IC2.19 (~{OE2}), J2.4, J3.4, J4.4, J5.4, J6.4, J7.4, J8.4, J9.4
- net +5V_Z: now reaches C5.1, J1.1 (VCC), PS1.1 (+VIN)
- net +5V_Z: now also C7.1, C8.1, D1.1 (K), IC1.20 (VCC), IC2.20 (VCC), J2.1, J3.1, J4.1, J5.1, J6.1, J7.1, J8.1, J9.1
- net Z_Out_DCC_Signal_A: now reaches U1.4 (IO4)
- net Z_Out_DCC_Signal_A: now also IC1.2 (A1), IC1.3 (A2), IC1.4 (A3), IC1.5 (A4), IC1.6 (A5), IC1.7 (A6), IC1.8 (A7), IC1.9 (A8)
- net Z_Out_DCC_Signal_B: now reaches U1.5 (IO5)
- net Z_Out_DCC_Signal_B: now also IC2.2 (A1), IC2.3 (A2), IC2.4 (A3), IC2.5 (A4), IC2.6 (A5), IC2.7 (A6), IC2.8 (A7), IC2.9 (A8)
- new net DCC_Signal_A_1: IC1.18 (Y1), J2.2
- new net DCC_Signal_A_2: IC1.17 (Y2), J3.2
- new net DCC_Signal_A_3: IC1.16 (Y3), J4.2
- new net DCC_Signal_A_4: IC1.15 (Y4), J5.2
- new net DCC_Signal_A_5: IC1.14 (Y5), J6.2
- new net DCC_Signal_A_6: IC1.13 (Y6), J7.2
- new net DCC_Signal_A_7: IC1.12 (Y7), J8.2
- new net DCC_Signal_A_8: IC1.11 (Y8), J9.2
- new net DCC_Signal_B_1: IC2.18 (Y1), J2.3
- new net DCC_Signal_B_2: IC2.17 (Y2), J3.3
- new net DCC_Signal_B_3: IC2.16 (Y3), J4.3
- new net DCC_Signal_B_4: IC2.15 (Y4), J5.3
- new net DCC_Signal_B_5: IC2.14 (Y5), J6.3
- new net DCC_Signal_B_6: IC2.13 (Y6), J7.3
- new net DCC_Signal_B_7: IC2.12 (Y7), J8.3
- new net DCC_Signal_B_8: IC2.11 (Y8), J9.3
Other:
- moved on the sheet: C1, C2, C3, C4, C5, PS1, R1, R2, SW1, SW2, U1

Commit message: hardware update push
Parts:
- removed D1: SMAJ5.0A, SYNCHRO_Library:DIOM5226X243N, symbol SYNCHRO_Library:SMAJ5.0A
- added C10, C11, C9: 10uF, Capacitor_SMD:C_1210_3225Metric_Pad1.33x2.70mm_HandSolder, symbol Device:C
- added C12: 22uF, Capacitor_SMD:C_1210_3225Metric_Pad1.33x2.70mm_HandSolder, symbol Device:C
- added D1: PMEG3010ER, Diode_SMD:Nexperia_CFP3_SOD-123W, symbol Device:D_Schottky
- added D2, D3, D4, D5, D6, D7: LED, LED_THT:LED_D5.0mm, symbol Device:LED
- added IC3: AZ1117CH-3.3TRG1, SYNCHRO_Library:SOT230P700X180-4N, symbol SYNCHRO_Library:AZ1117CH-3.3TRG1
- added J10: 694106301002, SYNCHRO_Library:694106301002, symbol SYNCHRO_Library:694106301002
- added J11: Conn_01x06, symbol Connector_Generic:Conn_01x06
- added PS2: R-78E5.0-1.0, SYNCHRO_Library:R78E5010, symbol SYNCHRO_Library:R-78E5.0-1.0
- added R10, R11, R7, R8, R9: 220, Resistor_SMD:R_0805_2012Metric_Pad1.20x1.40mm_HandSolder, symbol Device:R
- added R12: 470, Resistor_SMD:R_0805_2012Metric_Pad1.20x1.40mm_HandSolder, symbol Device:R
- added R3, R4, R5, R6: 10k, Resistor_SMD:R_0805_2012Metric_Pad1.20x1.40mm_HandSolder, symbol Device:R
- added SW3, SW4, SW5, SW6: SW_Push, Button_Switch_THT:SW_PUSH_6mm, symbol Switch:SW_Push
Connections:
- net +3.3V: now also D1.1 (K), R11.2, R3.2, R4.2, R5.2, R6.2
- net +5V_Z: now also C9.1, PS2.3 (+VOUT), R12.2; no longer C5.1, J1.1 (VCC), PS1.1 (+VIN)
- net GND: now also C10.2, C11.2, C12.2, C9.2, D2.1 (K), D3.1 (K), D4.1 (K), D5.1 (K), D6.1 (K), D7.1 (K), IC3.1 (GND), J10.2 (GND_1), J10.3 (GND_2), PS2.2 (GND), SW3.1, SW4.1, SW5.1, SW6.1
- net IO17: now reaches U1.10 (IO17)
- net IO17: now also J11.4 (Pin_4)
- net IO18: now reaches U1.11 (IO18)
- net IO18: now also J11.5 (Pin_5)
- net IO8: now reaches U1.12 (IO8)
- net IO8: now also R5.1, SW5.2
- net IO9: now reaches U1.17 (IO9)
- net IO9: now also R6.1, SW6.2
- net IO10: now reaches U1.18 (IO10)
- net IO10: now also R7.2
- net IO11: now reaches U1.19 (IO11)
- net IO11: now also R8.2
- net IO12: now reaches U1.20 (IO12)
- net IO12: now also R9.2
- net IO13: now reaches U1.21 (IO13)
- net IO13: now also R10.2
- net IO14: now reaches U1.22 (IO14)
- net IO14: now also J11.1 (Pin_1)
- net IO21: now reaches U1.23 (IO21)
- net IO21: now also J11.6 (Pin_6)
- net IO6: now reaches U1.6 (IO6)
- net IO6: now also R3.1, SW3.2
- net IO7: now reaches U1.7 (IO7)
- net IO7: now also R4.1, SW4.2
- net IO15: now reaches U1.8 (IO15)
- net IO15: now also J11.2 (Pin_2)
- net IO16: now reaches U1.9 (IO16)
- net IO16: now also J11.3 (Pin_3)
- new net: D2.2 (A), R7.1
- new net: C12.1, D1.2 (A), IC3.2 (OUTPUT), IC3.4 (VOUT)
- new net: C11.1, IC3.3 (INPUT), J1.1 (VCC)
- new net: D4.2 (A), R9.1
- new net: C10.1, C5.1, J10.1 (POWER), PS1.1 (+VIN), PS2.1 (+VIN)
- new net: D6.2 (A), R11.1
- new net: D7.2 (A), R12.1
- new net: D5.2 (A), R10.1
- new net: D3.2 (A), R8.1
Other:
- moved on the sheet: C1, C2, C5, C6, J1, PS1

Commit message: Zentrale Layout V1.0 finalisierung
Parts:
- removed J11: Conn_01x06, symbol Connector_Generic:Conn_01x06
Connections:
- net IO14: no longer names the net of U1.22 (IO14)
- net IO15: no longer names the net of U1.8 (IO15)
- net IO16: no longer names the net of U1.9 (IO16)
- net IO17: no longer names the net of U1.10 (IO17)
- net IO18: no longer names the net of U1.11 (IO18)
- net IO21: no longer names the net of U1.23 (IO21)
